File: design/powersupply/Senior Design Power PCB.sch (KiCad schematic (older format))
At the start: 10 parts, among them U1 INA226, U2 LM2596SX-5

Commit message: updated board layout
Parts:
- C1: value 680uF 35v (Panasonic FK) -> 470 uF 16v
- C2: value 680uF 35v (Panasonic FK) -> 220 uF 10v
- L1: value 33 uH -> 22 uH
Changed lines of the file:
@@
 P 7200 3600
 F 0 "L1" H 7200 3700 50  0000 C CNN
-F 1 "33 uH" H 7200 3550 50  0000 C CNN
+F 1 "22 uH" H 7200 3550 50  0000 C CNN
 F 2 "" H 7200 3600 50  0001 C CNN
 F 3 "~" H 7200 3600 50  0001 C CNN
@@
 U 1 1 5D7B82A7
 P 7550 3850
-F 0 "C2" H 7500 3600 50  0000 L CNN
-F 1 "680uF 35v (Panasonic FK)" H 7050 3500 50  0000 L CNN
+F 0 "C2" H 7600 4000 50  0000 L CNN
+F 1 "220 uF 10v" H 7300 3500 50  0000 L CNN
 F 2 "" H 7550 3850 50  0001 C CNN
 F 3 "~" H 7550 3850 50  0001 C CNN
@@
 U 1 1 5D7B7A85
 P 5350 3850
-F 0 "C1" H 5300 3600 50  0000 L CNN
-F 1 "680uF 35v (Panasonic FK)" H 5100 3500 50  0000 L CNN
+F 0 "C1" H 5200 4000 50  0000 L CNN
+F 1 "470 uF 16v" H 5100 3500 50  0000 L CNN
 F 2 "" H 5350 3850 50  0001 C CNN
 F 3 "~" H 5350 3850 50  0001 C CNN
