File: design/schematic/schematic.sch (KiCad schematic (older format))
At the start: 43 parts, among them M1 Drive Motor, M2 Steering Servo, P1 Raspberry Pi 4, Q1 IRF250, SW1 Logic Power, SW1 Pi Shutdown, SW1 SW_SPST, SW2 Reset, SW2 SW_SPST, U1 DC-DC Converter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

Commit message: added full schematic
Parts:
- M?: symbol Custom:ESC -> schematic-rescue:ESC-Custom
- U1: symbol Custom:Level_Converter -> schematic-rescue:Level_Converter-Custom
- U4: symbol Custom:SSD1386 -> schematic-rescue:SSD1386-Custom
Changed lines of the file:
@@
 $EndComp
 $Comp
-L Custom:SSD1386 U4
+L schematic-rescue:SSD1386-Custom U4
 U 1 1 5DFA12B3
 P 6050 3950
@@
 	6650 4550 6650 4650
 $Comp
-L Custom:Level_Converter U1
+L schematic-rescue:Level_Converter-Custom U1
 U 1 1 5DFAF6AB
 P 6050 2050
@@
 	13150 3650 13450 3650
 $Comp
-L Custom:ESC M?
+L schematic-rescue:ESC-Custom M?
 U 1 1 5E0DD40B
 P 12600 3800
@@
 Wire Wire Line
 	10750 3600 12250 3600
+Text Label 3700 6550 0    59   ~ 0
+SDA
+Text Label 3700 6650 0    59   ~ 0
+SCL
 Wire Bus Line
 	4100 5750 6500 5750
@@
 Wire Bus Line
 	8500 5000 9350 5000
-Text Label 3700 6550 0    59   ~ 0
-SDA
-Text Label 3700 6650 0    59   ~ 0
-SCL
 $EndSCHEMATC
